Commit message: fix: 修复导航启动 URDF/桥接配置 + 相机图像 180° 倒置
- dog_brain: navigation_launch.py 同步 mapping_launch 的两处修复——
  robot_description 用 Command('cat')+ParameterValue(str) 读入 URDF 内容，
  lcm_bridge 不再把扁平 bridge_params.yaml 当 ROS2 params 传
- dog_description: camera_joint 朝向 rpy 由 0 改为 180° roll(绕X)，
  修正 rviz2 中 D435i 相机图像倒置 180°；add_sensor_frames.py 同步该朝向

File: src/dog_description/urdf/dog.urdf (robot description, URDF)
Before this commit: robot new_z1w, 19 links, 18 joints
Joints:
- joint camera_joint: origin xyz=0.35 0 0.08 rpy=0 0 0 -> xyz=0.35 0 0.08 rpy=3.141592653589793 0 0

Commit message: feat(navigation): Nav2 导航栈全链路联调修复
Nav2 激活与插件修复 (nav2_3d_params.yaml):
- 插件类名按 pluginlib ID 修正: navfn/behaviors/bt_navigator 用斜杠, waypoint_follower 用双冒号
- 移除新版 Humble 已删的 BT 库条目 (always_failure/remove_in_collision_goals)
- 雷达观测源 /livox/lidar(CustomMsg) 改用 /cloud_registered_body(PointCloud2, frame=base_link)
- voxel origin_z 0.0 -> -0.30 解决传感器原点 raytrace 越界

新增 pcd_to_map_node.py: PCD 3D 地图投影 2D OccupancyGrid 发 /map (transient_local), 供 static_layer
global_map_publisher.py: 修复 points.tolist() 性能灾难, 一次性缓存 PointCloud2 (tobytes)
publish_initial_pose.py: 修复 Point/Quaternion 位置参数 TypeError + 循环发布确保 DDS 送达
navigation_launch.py + CMakeLists.txt: 集成 pcd_to_map 节点

其余累积修复:
- pub_handler.cpp: Livox 时间戳软件补偿补丁 (GetEthPacketTimestamp, min-delay 滤波)
- dog.urdf / mid360.yaml / lcm_bridge bridge_params.yaml 等配置修正
- global_localization/transform_fusion 执行权限

验证: Nav2 9 服务器全 active, ICP fitness=1.000, /map 523x338, /cmd_vel 通电

File: src/dog_description/urdf/dog.urdf (robot description, URDF)
Before this commit: robot new_z1w, 19 links, 18 joints
Joints:
- joint FL_hip_joint: axis 1 0 0 -> -1 0 0
- joint FR_hip_joint: axis 1 0 0 -> -1 0 0
- joint RL_hip_joint: axis 1 0 0 -> -1 0 0
- joint RR_hip_joint: axis 1 0 0 -> -1 0 0

Commit message: fix: 传感器优化 - step_detector 降频 10Hz + OPENBLAS_NUM_THREADS=1、狗体点云屏蔽、URDF 外参修正 livox 0.45m/camera 0.50m

File: src/dog_description/urdf/dog.urdf (robot description, URDF)
Before this commit: robot new_z1w, 19 links, 18 joints
Joints:
- joint camera_joint: origin xyz=0.35 0 0.08 rpy=3.141592653589793 0 0 -> xyz=0.50 0 0.07 rpy=3.141592653589793 0 0
- joint livox_joint: origin xyz=0.30 0 0.15 rpy=0 0 0 -> xyz=0.45 0 0.14 rpy=0 0 0
